Commit message: 记录履带实测尺寸并增加开环试车入口
按实测机身尺寸和履带中心距更新模型；新增仅供驱动联调的双路原始电机命令入口，保留正常速度控制与建图导航锁定。补充试车、超时停车和参数排障说明，并验证伪终端命令链路。

File: src/kiwi_slam/urdf/tracked.urdf.xacro (robot description, xacro)
@@ -24,5 +24,5 @@
   <joint name="left_track_joint" type="fixed">
     <parent link="base_link"/><child link="left_track"/>
-    <origin xyz="0 ${model['base_width_m'] / 2 + model['track_width_m'] / 2} ${-model['base_height_m'] / 2}"/>
+    <origin xyz="0 ${hardware['tracked_base_node']['ros__parameters']['track_separation_m'] / 2} ${-model['base_height_m'] / 2}"/>
   </joint>
   <link name="right_track">
@@ -31,5 +31,5 @@
   <joint name="right_track_joint" type="fixed">
     <parent link="base_link"/><child link="right_track"/>
-    <origin xyz="0 ${-model['base_width_m'] / 2 - model['track_width_m'] / 2} ${-model['base_height_m'] / 2}"/>
+    <origin xyz="0 ${-hardware['tracked_base_node']['ros__parameters']['track_separation_m'] / 2} ${-model['base_height_m'] / 2}"/>
   </joint>
   <link name="lidar_link"/>
